File: StarvingStudent.brd (EAGLE design)
At the start: 99.9 x 75.2 mm, 38 parts, among them J1 1X2-3.5MM, J2 1X3-3.5MM, J3 1X3-3.5MM, J4 1X3-3.5MM, J5 1X3-3.5MM

Commit message: Added drawings document and added drill legend to board file.
Parts:
- added DRILEGEND: (no value), drilegend:DRILEGEND
Other:
- board text added: "01-16"
- board text added: "01-20"
- board text added: "LAYER-STACK"
